File: orthoProject75.sch (KiCad schematic (older format))
At the start: 151 parts, among them SW1 SW_Push

Commit message: Added 5k1 resistors to type-c CC pins
Parts:
- removed D? (x75): D_ALT, symbol D_ALT
- removed SW1, SW? (x74): SW_Push, symbol SW_Push
- removed U?: STM32F072C(8-B)Tx, LQFP48, symbol STM32F072C(8-B)Tx
- added C1: 4u7, Capacitor_SMD:C_0402_1005Metric, symbol Device:C_Small
- added C2, C3, C4, C5: 100n, Capacitor_SMD:C_0402_1005Metric, symbol Device:C_Small
- added C6, C7: 1u, Capacitor_SMD:C_0402_1005Metric, symbol Device:C_Small
- added C8, C9: 30p, Capacitor_SMD:C_0402_1005Metric, symbol Device:C_Small
- added FB1: 100R, Inductor_SMD:L_0805_2012Metric_Pad1.15x1.40mm_HandSolder, symbol Device:Ferrite_Bead
- added H1, H10, H11, H12, H2, H3, H4, H5, H6, H7, H8, H9: MountingHole_Pad, MountingHole:MountingHole_2.7mm_M2.5_Pad_Via, symbol Mechanical:MountingHole_Pad
- added J1: CONN_LCD, macropad:Lolin_TFT_2.4, symbol Connector:Conn_01x12_Male
- added J2: TC2050-IDC, Connector:Tag-Connect_TC2050-IDC-FP_2x05_P1.27mm_Vertical, symbol Connector_Generic:Conn_02x05_Counter_Clockwise
- added J3: USB_C_Receptacle_USB2.0, Connector_USB:USB_C_Receptacle_GCT_USB4085, symbol Connector:USB_C_Receptacle_USB2.0
- added JP1: SolderJumper_2_Open, Jumper:SolderJumper-2_P1.3mm_Open_RoundedPad1.0x1.5mm, symbol Jumper:SolderJumper_2_Open
- added LED1: LED, LED_SMD:LED_0603_1608Metric_Pad1.05x0.95mm_HandSolder, symbol Device:LED
- added R1, R2, R3: 1k5, Resistor_SMD:R_0805_2012Metric_Pad1.15x1.40mm_HandSolder, symbol Device:R_Small
- added RUSB1, RUSB2: 5k1, Resistor_SMD:R_0805_2012Metric_Pad1.15x1.40mm_HandSolder, symbol Device:R_Small
- added U1: XC6206P332MR, Package_TO_SOT_SMD:SOT-23, symbol Regulator_Linear:XC6206PxxxMR
- added U2: STM32F303RCTx, Package_QFP:LQFP-64_10x10mm_P0.5mm, symbol MCU_ST_STM32F3:STM32F303RCTx
- added U3: USBLC6-2SC6, Package_TO_SOT_SMD:SOT-23-6, symbol Power_Protection:USBLC6-2SC6
- added Y1: 32MHz, Crystal:Crystal_SMD_7050-4Pin_7.0x5.0mm, symbol Device:Crystal_GND24_Small
Connections:
- net labels added: +3.3V, +5V, Col0, GND, HSE_IN, HSE_OUT, LCD_CS, LCD_DC, LCD_LED, LCD_RST, NRST, Row0, SPI_MISO, SPI_MOSI, SPI_SCK, SWCLK, SWDIO, SWO, TS_BSY, TS_CS, UART_RX, UART_TX, USBD+, USBD-
- net labels removed: Col14, Col15
- wire segments 21 -> 101
- no-connect marks 0 -> 20
Other:
- note added: "Cl = 2 * (CLOAD_CRYSTAL - CPARASITIC)"
- note added: "Key matrices"
- note added: "LCD Connection"
- note added: "Left key matrix"
- note added: "MCU"
- note added: "SWD"
- note added: "USB and power"
